Commit message: Update baocao(1).urdf

File: baocao(1).urdf (robot description, URDF)
Before this commit: robot your_robot_name, 9 links, 8 joints
Links:
- link after_left_wheel: mass 2 -> 0.1
- link after_right_wheel: mass 2 -> 0.1
- link base_link: mass 25 -> 5
- link befor_left_wheel: mass 2 -> 0.1
- link befor_right_wheel: mass 2 -> 0.1
- link camera_link: mass 0.5 -> 0.1
- link lidar_link: mass 0.5 -> 0.1

Commit message: Update baocao(1).urdf

File: baocao(1).urdf (robot description, URDF)
Before this commit: robot your_robot_name, 9 links, 8 joints
Links:
- removed link cot
- removed link court
- link base_link: geometry collision mesh filename=package://baocao/src/meshes/base.stl scale=0.001 0.001 0.001; visual box size=0.4 0.4 0.1
Joints:
- removed joint cot_joint
- removed joint robot_to_court

Commit message: Update baocao(1).urdf

File: baocao(1).urdf (robot description, URDF)
Before this commit: robot your_robot_name, 7 links, 6 joints
Links:
- link base_link: geometry collision mesh filename=package://baocao/src/meshes/base.stl scale=0.001 0.001 0.001; visual mesh filename=package://baocao/src/meshes/base.stl scale=0.001 0.001 0.001
